File: Hardware_STM32G431/_autosave-QuadEnv_Panel.kicad_pcb (KiCad board)
At the start: 2 copper layers, 20.3 x 128.5 mm, 16 parts

Commit message: Started creating firmware for STM32G431
Parts:
- moved kibuzzard-640B6CC5 0.25 mm to (65.4, 50.5)
Changed lines of the file:
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@@
     (fp_circle (center 0 0) (end 6 0) (layer "B.CrtYd") (width 0.05) (fill none))
     (pad "" np_thru_hole circle (at 0 0 180) (size 7 7) (drill 7) (layers F&B.Cu *.Mask))
-    (model "${CUSTOM_3D}/Sifam_Knob_Small_Tall_Unskirted.step"
+    (model "${CUSTOM_3D}/Sifam_Knob_Small_Unskirted.step"
       (offset (xyz 0 0 0))
       (scale (xyz 1 1 1))
@@
   )
   (footprint "kibuzzard-640B6CC5" (layer "B.Cu")
-    (at 65.15 50.5 180)
+    (at 65.4 50.5 180)
     (descr "Generated with KiBuzzard")
     (tags "kb_params=eyJBbGlnbm1lbnRDaG9pY2UiOiAiQ2VudGVyIiwgIkNhcExlZnRDaG9pY2UiOiAiWyIsICJDYXBSaWdodENob2ljZSI6ICIvIiwgIkZvbnRDb21ib0JveCI6ICJSb2JvdG8tQm9sZCIsICJIZWlnaHRDdHJsIjogIjIuNSIsICJMYXllckNvbWJvQm94IjogIkYuTWFzayIsICJNdWx0aUxpbmVUZXh0IjogIkEiLCAiUGFkZGluZ0JvdHRvbUN0cmwiOiAiMyIsICJQYWRkaW5nTGVmdEN0cmwiOiAiMTAiLCAiUGFkZGluZ1JpZ2h0Q3RybCI6ICIyMCIsICJQYWRkaW5nVG9wQ3RybCI6ICIzIiwgIldpZHRoQ3RybCI6ICIifQ==")
@@
     (fp_circle (center 0 0) (end 6 0) (layer "B.CrtYd") (width 0.05) (fill none))
     (pad "" np_thru_hole circle (at 0 0 180) (size 7 7) (drill 7) (layers F&B.Cu *.Mask))
-    (model "${CUSTOM_3D}/Sifam_Knob_Small_Tall_Unskirted.step"
+    (model "${CUSTOM_3D}/Sifam_Knob_Small_Unskirted.step"
       (offset (xyz 0 0 0))
       (scale (xyz 1 1 1))
@@
     (fp_circle (center 0 0) (end 6 0) (layer "B.CrtYd") (width 0.05) (fill none))
     (pad "" np_thru_hole circle (at 0 0 180) (size 7 7) (drill 7) (layers *.Cu *.Mask))
-    (model "${CUSTOM_3D}/Sifam_Knob_Small_Tall_Unskirted.step"
+    (model "${CUSTOM_3D}/Sifam_Knob_Small_Unskirted.step"
       (offset (xyz 0 0 0))
       (scale (xyz 1 1 1))
@@
     (fp_circle (center 0 0) (end 6 0) (layer "B.CrtYd") (width 0.05) (fill none))
     (pad "" np_thru_hole circle (at 0 0 180) (size 7 7) (drill 7) (layers F&B.Cu *.Mask))
-    (model "${CUSTOM_3D}/Sifam_Knob_Small_Tall_Unskirted.step"
+    (model "${CUSTOM_3D}/Sifam_Knob_Small_Unskirted.step"
       (offset (xyz 0 0 0))
       (scale (xyz 1 1 1))
@@
   (gr_rect (start 69.8 84) (end 59.4 98) (layer "B.Cu") (width 0.15) (fill solid))
   (gr_circle (center 59.4 54) (end 66.4 54) (layer "B.Cu") (width 0.15) (fill solid))
-  (gr_circle (center 59.2 110) (end 52.2 110) (layer "B.Cu") (width 0.15) (fill solid))
-  (gr_circle (center 59.2 72) (end 52.2 72) (layer "B.Cu") (width 0.15) (fill solid))
-  (gr_circle (center 59.6 91) (end 66.6 91) (layer "B.Cu") (width 0.15) (fill solid))
+  (gr_circle (center 59.4 110) (end 52.4 110) (layer "B.Cu") (width 0.15) (fill solid))
+  (gr_circle (center 59.4 72) (end 52.4 72) (layer "B.Cu") (width 0.15) (fill solid))
+  (gr_circle (center 59.4 91) (end 66.4 91) (layer "B.Cu") (width 0.15) (fill solid))
   (gr_rect (start 49 79) (end 59.4 65) (layer "B.Cu") (width 0.15) (fill solid))
   (gr_rect (start 69.6 47) (end 59.2 61) (layer "B.Cu") (width 0.15) (fill solid))
@@
       )
     )
-  )
-  (zone (net 0) (net_name "") (layer "B.Cu") (hatch edge 0.508)
-    (priority 1)
-    (connect_pads (clearance 0.508))
-    (min_thickness 0.254) (filled_areas_thickness no)
-    (fill yes (thermal_gap 0.508) (thermal_bridge_width 0.508))
-    (polygon
-      (pts
-        (xy 97.2 41.528869)
-        (xy 75 41.528869)
-        (xy 75 31.8)
-        (xy 97.2 31.8)
-      )
-    )
