File: Hardware/QuadEnv_Controls_2.kicad_pcb (KiCad board)
At the start: 2 copper layers, 18.8 x 110 mm, 15 parts, among them J1 Conn_01x08_Male, J2 Conn_01x04_Male, J3 Conn_01x05_Male, J4 Conn_01x04_Male, J5 Gate_In, J6 Env_Out

Commit message: Updated to version 2 of panel
Parts:
- J1: value Conn_01x08_Male -> Conn_01x08; footprint Connector_PinHeader_2.54mm:PinHeader_1x08_P2.54mm_Vertical -> Connector_PinSocket_2.54mm:PinSocket_1x08_P2.54mm_Vertical
- J2, J4: value Conn_01x04_Male -> Conn_01x04; footprint Connector_PinHeader_2.54mm:PinHeader_1x04_P2.54mm_Vertical -> Connector_PinSocket_2.54mm:PinSocket_1x04_P2.54mm_Vertical
- J3: value Conn_01x05_Male -> Conn_01x05; footprint Connector_PinHeader_2.54mm:PinHeader_1x05_P2.54mm_Vertical -> Connector_PinSocket_2.54mm:PinSocket_1x05_P2.54mm_Vertical
- moved D5 7.77 mm to (52.7, 97.4), turned to 90 degrees
Routing:
- net /Mode_Led: track 28.4 -> 17.3 mm
- net /Release_Pot: track 35.4 -> 28.2 mm

Commit message: Completed v2 design
Parts:
- moved D5 0.20 mm to (52.5, 97.4)
Changed lines of the file:
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@@
   )
   (footprint "Custom_Footprints:LED_D3.0mm" (layer "B.Cu")
-    (at 52.7 97.4 90)
+    (at 52.5 97.4 90)
     (descr "LED, diameter 3.0mm, 2 pins")
     (tags "LED diameter 3.0mm 2 pins")
@@
   (segment (start 64.2 143.7) (end 63.5 143) (width 0.25) (layer "F.Cu") (net 18))
   (segment (start 64.2 151.72) (end 64.2 143.7) (width 0.25) (layer "F.Cu") (net 18))
-  (segment (start 50.9 94.33) (end 50.9 81.38) (width 0.25) (layer "F.Cu") (net 27))
   (segment (start 50.9 81.38) (end 52.2 80.08) (width 0.25) (layer "F.Cu") (net 27))
-  (segment (start 52.7 96.13) (end 50.9 94.33) (width 0.25) (layer "F.Cu") (net 27))
+  (segment (start 50.9 94.53) (end 50.9 81.38) (width 0.25) (layer "F.Cu") (net 27))
+  (segment (start 52.5 96.13) (end 50.9 94.53) (width 0.25) (layer "F.Cu") (net 27))
   (segment (start 56.9 84) (end 55.52 82.62) (width 0.25) (layer "B.Cu") (net 28))
   (segment (start 55.52 82.62) (end 52.2 82.62) (width 0.25) (layer "B.Cu") (net 28))
