File: Hardware/QuadEnv_Panel_2.kicad_pcb (KiCad board)
At the start: 2 copper layers, 20.3 x 128.5 mm, 17 parts

Commit message: Completed v2 design
Parts:
- removed kibuzzard-64E1F58E: G***, kibuzzard-64E1F58E
- removed kibuzzard-64E1F613: G***, kibuzzard-64E1F613
- removed kibuzzard-64E1F644: G***, kibuzzard-64E1F644
- added kibuzzard-64E3524E: G***, kibuzzard-64E3524E, B.Cu at (67.9, 54.0)
- added kibuzzard-64E35286: G***, kibuzzard-64E35286, B.Cu at (51.0, 72.0)
- added kibuzzard-64E35296: G***, kibuzzard-64E35296, B.Cu at (50.9, 110.0)
